File: PNP.brd (EAGLE design)
At the start: 65.8 x 73.3 mm, 37 parts, among them IC1 AT90CAN-A, J3 PNPINTERFACE, J5 J5, U11 SCHMITT, U2 MCP2551SN, U3 TPIC8101, U4 VND5N07, U5 VND5N07, U6 VNS3NV04D, Y1 16MHz

Commit message: opened with latest eagle, also have some changes still floating on my system at home, commit them all so I remove the local copy
Parts:
- added C10, C11, C13, C14: 100nF, PNP:0805
- added U1: ST232TSSOP16, PNP:TSSOP16
- moved R3 62.7 mm to (43.4, 31.8), turned to 270 degrees
- moved R2 62.1 mm to (45.5, 31.8), turned to 270 degrees
- moved JTAG 38.4 mm to (6.60, 40.4)
- moved C17 17.8 mm to (21.2, 62.5)
- moved Y1 17.5 mm to (20.6, 66.5)
- moved C16 16.5 mm to (24.8, 62.3)
- moved C2 16.2 mm to (29.7, 62.2)
- moved R7 15.8 mm to (29.0, 33.5), turned to 0 degrees
- moved C1 15.5 mm to (32.3, 62.0)
- moved R1 15.5 mm to (35.6, 62.0)
- moved R5 15.4 mm to (40.1, 33.0), turned to 180 degrees
- moved L1 13.9 mm to (37.1, 36.7)
- moved C5 12.9 mm to (36.4, 40.2)
- moved IC1 12.6 mm to (31.0, 50.8)
- moved R6 12.4 mm to (35.6, 33.0), turned to 180 degrees
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Connections:
- new net N$10: C10.2, U1.3
- new net N$13: C11.1, U1.4
- new net N$17: C11.2, U1.5
- new net N$19: U1.7
- new net N$20: C13.2, U1.2
- new net N$21: C14.1, U1.6
- new net N$30: U1.14
- new net N$31: U1.13
- new net N$32: U1.8
- new net N$9: C10.1, U1.1
- new net RXD: IC1.2, U1.12
- new net RXD1: IC1.27, U1.9
- new net TXD: IC1.3, U1.11
- new net TXD1: IC1.28, U1.10
- net 5V: now also C13.1, U1.16
- net GND: now also C14.2, U1.15
- net N$5: now also U6.2
Other:
- board size 65.8 x 73.3 mm -> 62.7 x 66.9 mm
