File: PNP.sch (EAGLE design)
At the start: 37 parts, among them IC1 AT90CAN-A, J3 PNPINTERFACE, J5 J5, U11 SCHMITT, U2 MCP2551SN, U3 TPIC8101, U4 VND5N07, U5 VND5N07, U6 VNS3NV04D, Y1 16MHz

Commit message: opened with latest eagle, also have some changes still floating on my system at home, commit them all so I remove the local copy
Parts:
- added C10, C11, C13, C14: 100nF, PNP:CAP0805
- added U1: ST232TSSOP16, PNP:ST232TSSOP16
Connections:
- new net N$10: C10.2, U1.C1-
- new net N$13: C11.1, U1.C2+
- new net N$17: C11.2, U1.C2-
- new net N$19: U1.T2OUT
- new net N$20: C13.2, U1.V+
- new net N$21: C14.1, U1.V-
- new net N$30: U1.T1OUT
- new net N$31: U1.R1IN
- new net N$32: U1.R2IN
- new net N$9: C10.1, U1.C1+
- new net RXD: IC1.(RXD/PDI)PE0, U1.R1OUT
- new net RXD1: IC1.(RXD1/INT2)PD2, U1.R2OUT
- new net TXD: IC1.(TXD/PDO)PE1, U1.T1IN
- new net TXD1: IC1.(TXD1/INT3)PD3, U1.T2IN
- net 5V: now also C13.1, U1.VCC
- net GND: now also C14.2, U1.GND
- net N$5: now also U6.INPUT1
